Commit message: add node5 (node code on several files)

File: urdf/robot1.urdf (robot description, URDF)
Before this commit: robot rospibot_model_06, 5 links, 4 joints
Links:
- link base_link: geometry collision box size=0.287 0.19 0.003; collision sphere radius=0.033
- link left_wheel: geometry collision cylinder length=0.027 radius=0.033; visual cylinder length=0.01 radius=0.033
- link right_wheel: geometry collision cylinder length=0.027 radius=0.033; visual cylinder length=0.01 radius=0.033
Joints:
- joint joint_left_wheel: origin xyz=0 0.095 0.032 rpy=0 0 0 -> xyz=0 0.095 0.033 rpy=0 0 0
- joint joint_right_wheel: origin xyz=0 -0.095 0.032 rpy=0 0 0 -> xyz=0 -0.095 0.033 rpy=0 0 0

Commit message: working m1p1 pkg before clean

File: urdf/robot1.urdf (robot description, URDF)
Before this commit: robot rospibot_model_06, 5 links, 4 joints
Links:
- removed link left_wheel
- removed link neato_laser
- removed link right_wheel
- added link neato; visual box size=0.05 0.015 0.03
- link base_link: geometry collision box size=0.28 0.18 0.003; collision sphere radius=0.032
Joints:
- removed joint joint_left_wheel
- removed joint joint_right_wheel
- joint joint_laser: child neato_laser -> neato
